Commit message: Renamed to match youbot link 0.

File: youbot_jaco_gazebo/youbot_jaco_gazebo/urdf/youbot_jaco.urdf.xacro (robot description, xacro)
@@ -33,10 +33,10 @@
     <origin xyz="-0.159 0 0.046" rpy="0 0 0" />
   </xacro:youbot_plate>
-  <link name="arm_mount" />
+  <link name="arm_link_0" />
   <joint name="arm_mount_joint" type="fixed">
     <parent link="base_link" />
-    <child link = "arm_mount" />
+    <child link = "arm_link_0" />
     <origin xyz="0.143 0 0.02" rpy="0 0 0" />
   </joint>
-  <xacro:j2n6s300  base_parent="arm_mount"/>
+  <xacro:j2n6s300  base_parent="arm_link_0"/>
 </robot>

Commit message: Add dummy link without inertia

File: youbot_jaco_gazebo/youbot_jaco_gazebo/urdf/youbot_jaco.urdf.xacro (robot description, xacro)
@@ -22,4 +22,9 @@
   <!-- <xacro:include filename="$(find kinova_description)/urdf/j2n6s300.xacro"/> -->
   <!-- Now we can start using the macros xacro:included above to define the actual youbot -->
+  <link name="dummy"></link>
+  <joint name="dummy_joint" type="fixed">
+    <parent link="dummy"/>
+    <child link="base_footprint"/>
+  </joint>
   <xacro:youbot_base name="base"/>
   <xacro:youbot_plate name="plate" parent="base_link">

Commit message: Rename dummy link to robot

File: youbot_jaco_gazebo/youbot_jaco_gazebo/urdf/youbot_jaco.urdf.xacro (robot description, xacro)
@@ -22,7 +22,7 @@
   <!-- <xacro:include filename="$(find kinova_description)/urdf/j2n6s300.xacro"/> -->
   <!-- Now we can start using the macros xacro:included above to define the actual youbot -->
-  <link name="dummy"></link>
-  <joint name="dummy_joint" type="fixed">
-    <parent link="dummy"/>
+  <link name="robot"></link>
+  <joint name="robot_joint" type="fixed">
+    <parent link="robot"/>
     <child link="base_footprint"/>
   </joint>
